Commit message: Update robot.xacro

File: robot.xacro (robot description, xacro)
@@ -2,9 +2,9 @@
 <robot xmlns:xacro="http://www.ros.org/wiki/xacro" name="robot">
 	   <!-- This first link called "world" is empty -->
-    <link name="world"></link>
+    <link name="my world"></link>
         <!-- The base origin is offset from the world origin. -->
     <joint name="base_joint" type="floating">
         <origin xyz="0 0 0" rpy="0 0 0"/>
-        <parent link="world"/>
+        <parent link="my world"/>
         <child link="cube_frame"/>
     </joint>

Commit message: Update robot.xacro

File: robot.xacro (robot description, xacro)
@@ -1,12 +1,12 @@
 <?xml version="1.0"?>
 <robot xmlns:xacro="http://www.ros.org/wiki/xacro" name="robot">
-	   <!-- This first link called "world" is empty -->
-    <link name="my world"></link>
-        <!-- The base origin is offset from the world origin. -->
-    <joint name="base_joint" type="floating">
-        <origin xyz="0 0 0" rpy="0 0 0"/>
-        <parent link="my world"/>
-        <child link="cube_frame"/>
-    </joint>
+  <!-- This first link called "my world" is empty -->
+  <link name="my world"></link>
+  <!-- The base origin is offset from the world origin. -->
+  <joint name="base_joint" type="fixed">
+    <origin xyz="0 0 0" rpy="0 0 0"/>
+    <parent link="my world"/>
+    <child link="cube_frame"/>
+  </joint>
   <!-- Define properties for cube dimensions -->
   <xacro:property name="cube_length" value="1.0"/>    <!-- Length of the cube -->
@@ -16,8 +16,12 @@
   <xacro:property name="cube_y" value="0.0"/>
   <xacro:property name="cube_z" value="${cube_length / 2}"/> <!-- Half the cube length -->
-	<!-- Define properties for the disk dimensions -->
+  <!-- Define properties for the disk dimensions -->
   <xacro:property name="disk_radius" value="0.3"/>        <!-- Radius of the disk -->
   <xacro:property name="disk_thickness" value="0.1"/>     <!-- Thickness (height) of the disk -->
-	<!-- Macro for defining a visual edge -->
+  <!-- Defining colors -->
+  <xacro:property name="red" value="1 0 0 1"/>
+  <xacro:property name="yellow" value="1 0.5 0 1"/>
+  <xacro:property name="green" value="0 1 0 1"/>
+  <!-- Macro for defining a visual edge -->
   <xacro:macro name="visual_edge" params="edge x y z r p yaw">
     <visual name="${edge}">
@@ -33,5 +37,5 @@
   </xacro:macro>
   <!-- Macro for defining a disk link-->
-  <xacro:macro name="disk_link_macro" params="name xyz rpy radius thickness">
+  <xacro:macro name="disk_link_macro" params="name xyz rpy radius thickness rgba">
     <link name="${name}">
       <!-- Visual element for the disk -->
@@ -41,6 +45,6 @@
           <cylinder radius="${radius}" length="${thickness}"/>
         </geometry>
-        <material name="orange">
-          <color rgba="1 0.5 0 1"/> <!-- Orange color with RGBA values -->
+        <material name="color_${rgba}">
+          <color rgba="${rgba}"/> <!-- Color with RGBA values -->
         </material>
       </visual>
@@ -64,15 +68,15 @@
     <!-- Visual element for the main cube -->
     <xacro:visual_edge edge="ZXY" x="${(cube_length - cube_girth) / 2}" y="${cube_y+(cube_length - cube_girth) / 2}" z="${cube_z}" r="0" p="0" yaw="0"/>
-	 <xacro:visual_edge edge="ZX_Y" x="${-(cube_length - cube_girth) / 2}" y="${cube_y+(cube_length - cube_girth) / 2}" z="${cube_z}" r="0" p="0" yaw="0"/>
-	 <xacro:visual_edge edge="ZXY_" x="${(cube_length - cube_girth) / 2}" y="${cube_y-(cube_length - cube_girth) / 2}" z="${cube_z}" r="0" p="0" yaw="0"/>
-	 <xacro:visual_edge edge="ZX_Y_" x="${-(cube_length - cube_girth) / 2}" y="${cube_y-(cube_length - cube_girth) / 2}" z="${cube_z}" r="0" p="0" yaw="0"/>
-	 <xacro:visual_edge edge="XYZ" y="${(cube_length - cube_girth) / 2}" z="${cube_z+(cube_length/2)-(cube_girth/2)}" x="${cube_x}" r="0" p="${pi/2}" yaw="0"/>
-	 <xacro:visual_edge edge="XY_Z" y="${-(cube_length - cube_girth) / 2}" z="${cube_z+(cube_length/2)-(cube_girth/2)}" x="${cube_x}" r="0" p="${pi/2}" yaw="0"/>
-	 <xacro:visual_edge edge="XYZ_" y="${(cube_length - cube_girth) / 2}" z="${cube_z-(cube_length/2)+(cube_girth/2)}" x="${cube_x}" r="0" p="${pi/2}" yaw="0"/>
-	 <xacro:visual_edge edge="XY_Z_" y="${-(cube_length - cube_girth) / 2}" z="${cube_z-(cube_length/2)+(cube_girth/2)}" x="${cube_x}" r="0" p="${pi/2}" yaw="0"/>
-	 <xacro:visual_edge edge="YZX" z="${cube_z+(cube_length/2)-(cube_girth/2)}" x="${cube_x+(cube_length - cube_girth) / 2}" y="${cube_y}" r="${pi/2}" p="0" yaw="0"/>
-	 <xacro:visual_edge edge="YZ_X" z="${cube_z-(cube_length/2)+(cube_girth/2)}" x="${cube_x+(cube_length - cube_girth) / 2}" y="${cube_y}" r="${pi/2}" p="0" yaw="0"/>
-	 <xacro:visual_edge edge="YZX_" z="${cube_z+(cube_length/2)-(cube_girth/2)}" x="${cube_x-(cube_length - cube_girth) / 2}" y="${cube_y}" r="${pi/2}" p="0" yaw="0"/>
-	 <xacro:visual_edge edge="YZ_X_" z="${cube_z-(cube_length/2)+(cube_girth/2)}" x="${cube_x-(cube_length - cube_girth) / 2}" y="${cube_y}" r="${pi/2}" p="0" yaw="0"/>
+    <xacro:visual_edge edge="ZX_Y" x="${-(cube_length - cube_girth) / 2}" y="${cube_y+(cube_length - cube_girth) / 2}" z="${cube_z}" r="0" p="0" yaw="0"/>
+    <xacro:visual_edge edge="ZXY_" x="${(cube_length - cube_girth) / 2}" y="${cube_y-(cube_length - cube_girth) / 2}" z="${cube_z}" r="0" p="0" yaw="0"/>
+    <xacro:visual_edge edge="ZX_Y_" x="${-(cube_length - cube_girth) / 2}" y="${cube_y-(cube_length - cube_girth) / 2}" z="${cube_z}" r="0" p="0" yaw="0"/>
+    <xacro:visual_edge edge="XYZ" y="${(cube_length - cube_girth) / 2}" z="${cube_z+(cube_length/2)-(cube_girth/2)}" x="${cube_x}" r="0" p="${pi/2}" yaw="0"/>
+    <xacro:visual_edge edge="XY_Z" y="${-(cube_length - cube_girth) / 2}" z="${cube_z+(cube_length/2)-(cube_girth/2)}" x="${cube_x}" r="0" p="${pi/2}" yaw="0"/>
+    <xacro:visual_edge edge="XYZ_" y="${(cube_length - cube_girth) / 2}" z="${cube_z-(cube_length/2)+(cube_girth/2)}" x="${cube_x}" r="0" p="${pi/2}" yaw="0"/>
+    <xacro:visual_edge edge="XY_Z_" y="${-(cube_length - cube_girth) / 2}" z="${cube_z-(cube_length/2)+(cube_girth/2)}" x="${cube_x}" r="0" p="${pi/2}" yaw="0"/>
+    <xacro:visual_edge edge="YZX" z="${cube_z+(cube_length/2)-(cube_girth/2)}" x="${cube_x+(cube_length - cube_girth) / 2}" y="${cube_y}" r="${pi/2}" p="0" yaw="0"/>
+    <xacro:visual_edge edge="YZ_X" z="${cube_z-(cube_length/2)+(cube_girth/2)}" x="${cube_x+(cube_length - cube_girth) / 2}" y="${cube_y}" r="${pi/2}" p="0" yaw="0"/>
+    <xacro:visual_edge edge="YZX_" z="${cube_z+(cube_length/2)-(cube_girth/2)}" x="${cube_x-(cube_length - cube_girth) / 2}" y="${cube_y}" r="${pi/2}" p="0" yaw="0"/>
+    <xacro:visual_edge edge="YZ_X_" z="${cube_z-(cube_length/2)+(cube_girth/2)}" x="${cube_x-(cube_length - cube_girth) / 2}" y="${cube_y}" r="${pi/2}" p="0" yaw="0"/>
     <!-- Collision properties for the main link -->
     <collision name="collision">
@@ -90,7 +94,7 @@
   </link>
   <!-- Defining the Three Disks -->
-  <xacro:disk_link_macro name="disk_link_X" xyz="0 0 0" rpy="0 ${pi/2} 0" radius="${disk_radius}" thickness="${disk_thickness}"/>
-  <xacro:disk_link_macro name="disk_link_Y" xyz="0 0 0" rpy="${pi/2} 0 0" radius="${disk_radius}" thickness="${disk_thickness}"/>
-  <xacro:disk_link_macro name="disk_link_Z" xyz="0 0 0" rpy="0 0 0" radius="${disk_radius}" thickness="${disk_thickness}"/>
+  <xacro:disk_link_macro name="disk_link_X" xyz="0 0 0" rpy="0 ${pi/2} 0" radius="${disk_radius}" thickness="${disk_thickness}" rgba="${red}"/>
+  <xacro:disk_link_macro name="disk_link_Y" xyz="0 0 0" rpy="${pi/2} 0 0" radius="${disk_radius}" thickness="${disk_thickness}" rgba="${yellow}"/>
+  <xacro:disk_link_macro name="disk_link_Z" xyz="0 0 0" rpy="0 0 0" radius="${disk_radius}" thickness="${disk_thickness}" rgba="${green}"/>
   <!-- Joint between cube_frame and disk_links -->
   <joint name="cube_disk_joint_X" type="continuous">
@@ -98,49 +102,49 @@
     <parent link="cube_frame"/>
     <child link="disk_link_X"/>
-    <axis xyz="1 0 0"/> <!-- Rotation axis along the z-axis (adjust as needed) -->
-    <limit effort="1000.0" velocity="10.0"/> <!-- Joint effort and velocity limits (adjust as needed) -->
+    <axis xyz="1 0 0"/> <!-- Rotation axis along the x-axis -->
+    <limit effort="1000.0" velocity="1000.0"/> <!-- Joint effort and velocity limits -->
   </joint>
-   <joint name="cube_disk_joint_Y" type="continuous">
+  <joint name="cube_disk_joint_Y" type="continuous">
     <origin xyz="${cube_x} ${cube_y+(cube_length/2)-disk_thickness} ${cube_z}"/>
     <parent link="cube_frame"/>
     <child link="disk_link_Y"/>
-    <axis xyz="0 1 0"/> <!-- Rotation axis along the z-axis (adjust as needed) -->
-    <limit effort="1000.0" velocity="10.0"/> <!-- Joint effort and velocity limits (adjust as needed) -->
+    <axis xyz="0 1 0"/> <!-- Rotation axis along the y-axis -->
+    <limit effort="1000.0" velocity="1000.0"/> <!-- Joint effort and velocity limits -->
   </joint>
-   <joint name="cube_disk_joint_Z" type="continuous">
+  <joint name="cube_disk_joint_Z" type="continuous">
     <origin xyz="${cube_x} ${cube_y} ${cube_z+(cube_length/2)-disk_thickness}"/>
     <parent link="cube_frame"/>
     <child link="disk_link_Z"/>
-    <axis xyz="0 0 1"/> <!-- Rotation axis along the z-axis (adjust as needed) -->
-    <limit effort="1000.0" velocity="10.0"/> <!-- Joint effort and velocity limits (adjust as needed) -->
+    <axis xyz="0 0 1"/> <!-- Rotation axis along the z-axis -->
+    <limit effort="1000.0" velocity="1000.0"/> <!-- Joint effort and velocity limits -->
   </joint>
   <!-- JointController plugin to control the joint velocity (for cube_disk_joint_X)-->
   <gazebo>
-			<plugin filename="libignition-gazebo-joint-controller-system.so"
-			name="ignition::gazebo::systems::JointController">
-				<joint_name>cube_disk_joint_X</joint_name>
-				<topic>cmd_vel_r</topic>
-				<!-- PID controller for smooth velocity control -->
-				<use_force_commands>true</use_force_commands>
-				<p_gain>0.15</p_gain>
-			</plugin>
-			<!-- JointController plugin to control the joint velocity (for cube_disk_joint_y)-->
-			<plugin filename="libignition-gazebo-joint-controller-system.so"
-			name="ignition::gazebo::systems::JointController">
-				<joint_name>cube_disk_joint_Y</joint_name>
-				<topic>cmd_vel_y</topic>
-				<!-- PID controller for smooth velocity control -->
-				<use_force_commands>true</use_force_commands>
-				<p_gain>0.15</p_gain>
-			</plugin>
-			<!-- JointController plugin to control the joint velocity (for cube_disk_joint_Z)-->
-			<plugin filename="libignition-gazebo-joint-controller-system.so"
-			name="ignition::gazebo::systems::JointController">
-				<joint_name>cube_disk_joint_Z</joint_name>
-				<topic>cmd_vel_g</topic>
-				<!-- PID controller for smooth velocity control -->
-				<use_force_commands>true</use_force_commands>
-				<p_gain>0.15</p_gain>
-			</plugin>
-	</gazebo>
+    <plugin filename="libignition-gazebo-joint-controller-system.so"
+            name="ignition::gazebo::systems::JointController">
+      <joint_name>cube_disk_joint_X</joint_name>
+      <topic>cmd_vel_r</topic>
+      <!-- PID controller for smooth velocity control -->
+      <use_force_commands>true</use_force_commands>
+      <p_gain>0.15</p_gain>
+    </plugin>
+    <!-- JointController plugin to control the joint velocity (for cube_disk_joint_Y)-->
+    <plugin filename="libignition-gazebo-joint-controller-system.so"
+            name="ignition::gazebo::systems::JointController">
+      <joint_name>cube_disk_joint_Y</joint_name>
+      <topic>cmd_vel_y</topic>
+      <!-- PID controller for smooth velocity control -->
+      <use_force_commands>true</use_force_commands>
+      <p_gain>0.15</p_gain>
+    </plugin>
+    <!-- JointController plugin to control the joint velocity (for cube_disk_joint_Z)-->
+    <plugin filename="libignition-gazebo-joint-controller-system.so"
+            name="ignition::gazebo::systems::JointController">
+      <joint_name>cube_disk_joint_Z</joint_name>
+      <topic>cmd_vel_g</topic>
+      <!-- PID controller for smooth velocity control -->
+      <use_force_commands>true</use_force_commands>
+      <p_gain>0.15</p_gain>
+    </plugin>
+  </gazebo>
 </robot>
